File: KiCad/uranus-fpga-board/fpga.kicad_sch (KiCad schematic)
At the start: 1 part, among them U1 XC7K325T-3FFG900E

Commit message: updated journal entries and BOM
Parts:
- added R13: 100 Ohm, symbol Device:R_Small
Connections:
- net GND: now reaches U1.A1 (GND)
- net GND: now also U1.A14 (GND), U1.A2 (GND), U1.A24 (GND), U1.A5 (GND), U1.A6 (GND), U1.A9 (GND), U1.AA1 (GND), U1.AA14 (GND), U1.AA2 (GND), U1.AA24 (GND), U1.AA5 (GND), U1.AA6 (GND), U1.AA7 (GND), U1.AB11 (GND), U1.AB21 (GND), U1.AB3 (GND), U1.AB4 (GND), U1.AC18 (GND), U1.AC28 (GND), U1.AC8 (GND), U1.AD15 (GND), U1.AD25 (GND), U1.AD5 (GND), U1.AE12 (GND), U1.AE2 (GND), U1.AE22 (GND), U1.AF19 (GND), U1.AF29 (GND), U1.AF9 (GND), U1.AG16 (GND), U1.AG26 (GND), U1.AG6 (GND), U1.AH13 (GND), U1.AH23 (GND), U1.AH3 (GND), U1.AJ10 (GND), U1.AJ20 (GND), U1.AJ30 (GND), U1.AK17 (GND), U1.AK27 (GND), U1.AK7 (GND), U1.B11 (GND), U1.B21 (GND), U1.B4 (GND), U1.B8 (GND), U1.B9 (GND), U1.C1 (GND), U1.C10 (VCCBATT_0), U1.C18 (GND), U1.C2 (GND), U1.C28 (GND), U1.C6 (GND), U1.C9 (GND), U1.D15 (GND), U1.D25 (GND), U1.D4 (GND), U1.D8 (GND), U1.D9 (GND), U1.E1 (GND), U1.E12 (GND), U1.E2 (GND), U1.E22 (GND), U1.E6 (GND), U1.E9 (GND), U1.F19 (GND), U1.F29 (GND), U1.F4 (GND), U1.F8 (GND), U1.F9 (GND), U1.G1 (GND), U1.G16 (GND), U1.G2 (GND), U1.G26 (GND), U1.G6 (GND), U1.G9 (GND), U1.H13 (GND), U1.H23 (GND), U1.H4 (GND), U1.H8 (GND), U1.H9 (GND), U1.J1 (GND), U1.J10 (GND), U1.J2 (GND), U1.J20 (GND), U1.J30 (GND), U1.J6 (GND), U1.J9 (GND), U1.K17 (GND), U1.K27 (GND), U1.K4 (GND), U1.K8 (GND), U1.K9 (GND), U1.L1 (GND), U1.L14 (GND), U1.L2 (GND), U1.L24 (GND), U1.L6 (GND), U1.L9 (GND), U1.M12 (GND), U1.M14 (GND), U1.M16 (GND), U1.M18 (GND), U1.M21 (GND), U1.M4 (GND), U1.M8 (GND), U1.M9 (GND), U1.N1 (GND), U1.N11 (GND), U1.N13 (GND), U1.N15 (GND), U1.N17 (GND), U1.N2 (GND), U1.N28 (GND), U1.N6 (GND), U1.N9 (GND), U1.P10 (GND), U1.P12 (GND), U1.P14 (GNDADC_0), U1.P16 (GND), U1.P18 (GND), U1.P25 (GND), U1.P4 (GND), U1.P8 (GND), U1.P9 (GND), U1.R1 (GND), U1.R11 (GND), U1.R13 (GND), U1.R17 (GND), U1.R2 (GND), U1.R22 (GND), U1.R6 (GND), U1.R9 (GND), U1.T10 (GND), U1.T12 (GND), U1.T16 (GND), U1.T18 (GND), U1.T19 (GND), U1.T29 (GND), U1.T4 (GND), U1.T8 (GND), U1.U1 (GND), U1.U11 (GND), U1.U13 (GND), U1.U17 (GND), U1.U2 (GND), U1.U26 (GND), U1.U6 (GND), U1.U9 (GND), U1.V10 (GND), U1.V12 (GND), U1.V14 (GND), U1.V16 (GND), U1.V18 (GND), U1.V23 (GND), U1.V4 (GND), U1.V8 (GND), U1.V9 (GND), U1.W1 (GND), U1.W11 (GND), U1.W13 (GND), U1.W15 (GND), U1.W17 (GND), U1.W2 (GND), U1.W20 (GND), U1.W30 (GND), U1.W6 (GND), U1.W9 (GND), U1.Y17 (GND), U1.Y27 (GND), U1.Y3 (GND), U1.Y4 (GND), U1.Y7 (GND), U1.Y8 (GND), U1.Y9 (GND)
- net +1V8_GTX: now reaches U1.B3 (MGTAVTT)
- net +1V8_GTX: now also U1.C5 (MGTAVTT), U1.D3 (MGTAVTT), U1.E5 (MGTAVTT), U1.F3 (MGTAVTT), U1.G5 (MGTAVTT), U1.H3 (MGTAVTT), U1.J5 (MGTAVTT), U1.K3 (MGTAVTT), U1.L5 (MGTAVTT), U1.M3 (MGTAVTT), U1.N5 (MGTAVTT), U1.P3 (MGTAVTT), U1.R5 (MGTAVTT), U1.T3 (MGTAVTT), U1.T7 (MGTVCCAUX), U1.U5 (MGTAVTT), U1.V3 (MGTAVTT), U1.V7 (MGTVCCAUX), U1.W5 (MGTAVTT), U1.W7 (MGTAVTTRCAL_115), R13.2
- net +1V05_GTX: now reaches U1.B7 (MGTAVCC)
- net +1V05_GTX: now also U1.D7 (MGTAVCC), U1.F7 (MGTAVCC), U1.H7 (MGTAVCC), U1.K7 (MGTAVCC), U1.M7 (MGTAVCC), U1.P7 (MGTAVCC)
- net +1V0: now reaches U1.N16 (VCCBRAM)
- net +1V0: now also U1.M11 (VCCINT), U1.M13 (VCCINT), U1.M15 (VCCINT), U1.M17 (VCCINT), U1.N10 (VCCINT), U1.N12 (VCCINT), U1.N14 (VCCINT), U1.N18 (VCCINT), U1.P11 (VCCINT), U1.P17 (VCCINT), U1.R10 (VCCINT), U1.R12 (VCCINT), U1.R16 (VCCBRAM), U1.R18 (VCCINT), U1.T11 (VCCINT), U1.T17 (VCCINT), U1.U10 (VCCINT), U1.U12 (VCCINT), U1.U16 (VCCBRAM), U1.U18 (VCCINT), U1.V17 (VCCINT), U1.W16 (VCCBRAM), U1.W18 (VCCINT)
- net +1V8: now reaches U1.P13 (VCCAUX)
- net +1V8: now also U1.P15 (VCCADC_0), U1.T13 (VCCAUX), U1.V11 (VCCAUX_IO_G0), U1.V13 (VCCAUX), U1.V15 (VCCAUX), U1.W10 (VCCAUX_IO_G0), U1.W12 (VCCAUX_IO_G0), U1.W14 (VCCAUX)
- net +2V5: now reaches U1.C13 (VCCO_18)
- net +2V5: now also U1.D10 (VCCO_18), U1.F14 (VCCO_18), U1.G11 (VCCO_18), U1.J15 (VCCO_18), U1.K12 (VCCO_18)
- net DQ56: now reaches U1.AA15 (IO_L20P_T3_32)
- net DM6: now reaches U1.AA18 (IO_L16P_T2_32)
- net DQ57: now reaches U1.AB15 (IO_L20N_T3_32)
- net DQ55: now reaches U1.AB17 (IO_L18P_T2_32)
- net DQ52: now reaches U1.AB18 (IO_L16N_T2_32)
- net DQ53: now reaches U1.AB19 (IO_L17P_T2_32)
- net DQ54: now reaches U1.AC19 (IO_L17N_T2_32)
- net DM7: now reaches U1.AE15 (IO_L19P_T3_32)
- net DQ24: now reaches U1.AF7 (IO_L20P_T3_34)
- net DM3: now reaches U1.AF8 (IO_L19P_T3_34)
- net DQ25: now reaches U1.AG7 (IO_L20N_T3_34)
- net DM2: now reaches U1.AH2 (IO_L16P_T2_34)
- net DQ21: now reaches U1.AJ1 (IO_L17P_T2_34)
- net DQ20: now reaches U1.AJ2 (IO_L16N_T2_34)
- net DQ23: now reaches U1.AJ3 (IO_L18P_T2_34)
- net DQ22: now reaches U1.AK1 (IO_L17N_T2_34)
- net at U1.W8 (MGTRREF_115): now also R13.1
- net A4: now reaches U1.AA13 (IO_L6P_T0_33)
- net A2: now reaches U1.AB10 (IO_L7P_T1_33)
- net A3: now reaches U1.AB13 (IO_L6N_T0_VREF_33)
- net A1: now reaches U1.AC10 (IO_L7N_T1_33)
- net BA0: now reaches U1.AC11 (IO_L9N_T1_DQS_33)
- net BA1: now reaches U1.AC12 (IO_L9P_T1_DQS_33)
- net DQ07: now reaches U1.AC7 (IO_L6P_T0_34)
- net DQ43: now reaches U1.AD19 (IO_L10P_T1_32)
- net A0: now reaches U1.AD8 (IO_L8P_T1_33)
- net RAS_N: now reaches U1.AD9 (IO_L10P_T1_33)
- net DQ09: now reaches U1.AE1 (IO_L8P_T1_34)
- net DQ39: now reaches U1.AE16 (IO_L6P_T0_32)
- net DQ44: now reaches U1.AE19 (IO_L10N_T1_32)
- net DQ12: now reaches U1.AE3 (IO_L10N_T1_34)
- net DQ11: now reaches U1.AE4 (IO_L10P_T1_34)
- net BA2: now reaches U1.AE8 (IO_L8N_T1_33)
- net CAS_N: now reaches U1.AE9 (IO_L10N_T1_33)
- net DQ10: now reaches U1.AF1 (IO_L8N_T1_34)
- net DQ08: now reaches U1.AF2 (IO_L7N_T1_34)
- net DM1: now reaches U1.AF3 (IO_L7P_T1_34)
- net DQ41: now reaches U1.AG19 (IO_L8P_T1_32)
- net DQS_N1: now reaches U1.AG3 (IO_L9N_T1_DQS_34)
- net DQS_P1: now reaches U1.AG4 (IO_L9P_T1_DQS_34)
- net DQ42: now reaches U1.AH19 (IO_L8N_T1_32)
- net DQS_P5: now reaches U1.AJ18 (IO_L9P_T1_DQS_32)
- net DM5: now reaches U1.AJ19 (IO_L7P_T1_32)
- net DQS_N5: now reaches U1.AK18 (IO_L9N_T1_DQS_32)
- net DQ40: now reaches U1.AK19 (IO_L7N_T1_32)
- net DQ51: now reaches U1.AD16 (IO_L14N_T2_SRCC_32)
- net DQ50: now reaches U1.AD17 (IO_L14P_T2_SRCC_32)
- net DQ48: now reaches U1.AD18 (IO_L13P_T2_MRCC_32)
- net CLK_P: now reaches U1.AE10 (IO_L14P_T2_SRCC_33)
- net WE_N: now reaches U1.AE11 (IO_L11P_T1_SRCC_33)
- net DQ49: now reaches U1.AE18 (IO_L13N_T2_MRCC_32)
- net DQ13: now reaches U1.AE5 (IO_L11P_T1_SRCC_34)
- net CLK_N: now reaches U1.AF10 (IO_L14N_T2_SRCC_33)
- net CS_N: now reaches U1.AF11 (IO_L11N_T1_SRCC_33)
- net DQ47: now reaches U1.AF17 (IO_L12P_T1_MRCC_32)
- net DQ45: now reaches U1.AF18 (IO_L11P_T1_SRCC_32)
- net DQ14: now reaches U1.AF5 (IO_L11N_T1_SRCC_34)
- net DQ15: now reaches U1.AF6 (IO_L12P_T1_MRCC_34)
- net REF_P: now reaches U1.AG10 (IO_L13P_T2_MRCC_33)
- net DQ46: now reaches U1.AG18 (IO_L11N_T1_SRCC_32)
- net DQS_P2: now reaches U1.AG2 (IO_L15P_T2_DQS_34)
- net RESET: now reaches U1.AG5 (IO_L12N_T1_MRCC_34)
- net DQS_N2: now reaches U1.AH1 (IO_L15N_T2_DQS_34)
- net REF_N: now reaches U1.AH10 (IO_L13N_T2_MRCC_33)
- net DQ16: now reaches U1.AH4 (IO_L13P_T2_MRCC_34)
- net DQ19: now reaches U1.AH5 (IO_L14N_T2_SRCC_34)
- net DQ18: now reaches U1.AH6 (IO_L14P_T2_SRCC_34)
- net DQ17: now reaches U1.AJ4 (IO_L13N_T2_MRCC_34)
- net CKE: now reaches U1.AJ9 (IO_L15P_T2_DQS_33)
- net ODT: now reaches U1.AK9 (IO_L15N_T2_DQS_33)
- net DQS_N6: now reaches U1.Y18 (IO_L15N_T2_DQS_32)
- net DQS_P6: now reaches U1.Y19 (IO_L15P_T2_DQS_32)
- net A5: now reaches U1.AA10 (IO_L5N_T0_33)
- net A6: now reaches U1.AA11 (IO_L5P_T0_33)
- net A12: now reaches U1.AA12 (IO_L1P_T0_33)
- net A10: now reaches U1.AA8 (IO_L2P_T0_33)
- net A11: now reaches U1.AB12 (IO_L1N_T0_33)
- net A9: now reaches U1.AB8 (IO_L2N_T0_33)
- net CK_P: now reaches U1.AB9 (IO_L3P_T0_DQS_33)
- net DQ02: now reaches U1.AC1 (IO_L2N_T0_34)
- net DQ01: now reaches U1.AC2 (IO_L2P_T0_34)
- net DQ04: now reaches U1.AC4 (IO_L4N_T0_34)
- net DQ03: now reaches U1.AC5 (IO_L4P_T0_34)
- net CK_N: now reaches U1.AC9 (IO_L3N_T0_DQS_33)
- net DQS_N0: now reaches U1.AD1 (IO_L3N_T0_DQS_34)
- net DQS_P0: now reaches U1.AD2 (IO_L3P_T0_DQS_34)
- net DQ00: now reaches U1.AD3 (IO_L1N_T0_34)
- net DM0: now reaches U1.AD4 (IO_L1P_T0_34)
- net DQ05: now reaches U1.AD6 (IO_L5P_T0_34)
- net DQ06: now reaches U1.AE6 (IO_L5N_T0_34)
- net DQ35: now reaches U1.AF15 (IO_L4P_T0_32)
- net DQ36: now reaches U1.AG14 (IO_L4N_T0_32)
- net DQ33: now reaches U1.AG15 (IO_L2P_T0_32)
- net DQ34: now reaches U1.AH15 (IO_L2N_T0_32)
- net DQS_P4: now reaches U1.AH16 (IO_L3P_T0_DQS_32)
- net DQ37: now reaches U1.AH17 (IO_L5P_T0_32)
- net DQS_N4: now reaches U1.AJ16 (IO_L3N_T0_DQS_32)
- net DQ38: now reaches U1.AJ17 (IO_L5N_T0_32)
- net DQ32: now reaches U1.AK15 (IO_L1N_T0_32)
- net DM4: now reaches U1.AK16 (IO_L1P_T0_32)
- net A7: now reaches U1.Y10 (IO_L4N_T0_33)
- net A8: now reaches U1.Y11 (IO_L4P_T0_33)
- net DQ61: now reaches U1.AA16 (IO_L23N_T3_32)
- net DQ60: now reaches U1.AA17 (IO_L23P_T3_32)
- net DQ58: now reaches U1.AC14 (IO_L22P_T3_32)
- net DQS_N7: now reaches U1.AC15 (IO_L21N_T3_DQS_32)
- net DQS_P7: now reaches U1.AC16 (IO_L21P_T3_DQS_32)
- net DQ59: now reaches U1.AD14 (IO_L22N_T3_32)
- net DQS_P3: now reaches U1.AH7 (IO_L21P_T3_DQS_34)
- net DQ26: now reaches U1.AJ6 (IO_L22P_T3_34)
- net DQS_N3: now reaches U1.AJ7 (IO_L21N_T3_DQS_34)
- net DQ28: now reaches U1.AJ8 (IO_L23P_T3_34)
- net DQ31: now reaches U1.AK4 (IO_L24N_T3_34)
- net DQ30: now reaches U1.AK5 (IO_L24P_T3_34)
- net DQ27: now reaches U1.AK6 (IO_L22N_T3_34)
- net DQ29: now reaches U1.AK8 (IO_L23N_T3_34)
- net DQ63: now reaches U1.Y15 (IO_L24N_T3_32)
- net DQ62: now reaches U1.Y16 (IO_L24P_T3_32)
Other:
- note added: "0.1%"
- moved on the sheet: U1E, U1F, U1G
